File: fonte.brd (EAGLE design)
At the start: 100 x 80 mm, 9 parts, among them T1 2N3904, X1 22-23-2021, X2 22-23-2021

Commit message: Add files via upload
Parts:
- R1: value 2k -> 5k6
- R2: value 4k7 -> 10k
- R4: value 200R -> 2k2
Changed lines of the file:
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@@
 <attribute name="VALUE" x="29.337" y="59.69" size="1.27" layer="27" ratio="10"/>
 </element>
-<element name="R2" library="pot" library_urn="urn:adsk.eagle:library:331" package="3RP/1610N" package3d_urn="urn:adsk.eagle:package:22726/1" value="4k7" x="40.64" y="46.99" smashed="yes" rot="R270">
+<element name="R2" library="pot" library_urn="urn:adsk.eagle:library:331" package="3RP/1610N" package3d_urn="urn:adsk.eagle:package:22726/1" value="10k" x="40.64" y="46.99" smashed="yes" rot="R270">
 <attribute name="NAME" x="46.355" y="55.245" size="1.27" layer="25" rot="R270"/>
 <attribute name="POPULARITY" value="8" x="26.67" y="25.4" size="1.778" layer="27" rot="R270" display="off"/>
@@
 <attribute name="VALUE" x="23.495" y="39.116" size="1.27" layer="27" ratio="10"/>
 </element>
-<element name="R4" library="rcl" library_urn="urn:adsk.eagle:library:334" package="0207/10" package3d_urn="urn:adsk.eagle:package:23491/2" value="200R" x="20.32" y="52.07" smashed="yes" rot="R270">
+<element name="R4" library="rcl" library_urn="urn:adsk.eagle:library:334" package="0207/10" package3d_urn="urn:adsk.eagle:package:23491/2" value="2k2" x="20.32" y="52.07" smashed="yes" rot="R270">
 <attribute name="NAME" x="21.844" y="55.118" size="1.27" layer="25" ratio="10" rot="R270"/>
 <attribute name="POPULARITY" value="81" x="20.32" y="52.07" size="1.778" layer="27" rot="R270" display="off"/>
@@
 <attribute name="VALUE" x="19.685" y="54.3306" size="1.27" layer="27" ratio="10" rot="R270"/>
 </element>
-<element name="R1" library="rcl" library_urn="urn:adsk.eagle:library:334" package="0207/10" package3d_urn="urn:adsk.eagle:package:23491/2" value="2k" x="40.64" y="60.96" smashed="yes" rot="R180">
+<element name="R1" library="rcl" library_urn="urn:adsk.eagle:library:334" package="0207/10" package3d_urn="urn:adsk.eagle:package:23491/2" value="5k6" x="40.64" y="60.96" smashed="yes" rot="R180">
 <attribute name="NAME" x="43.688" y="59.436" size="1.27" layer="25" ratio="10" rot="R180"/>
 <attribute name="POPULARITY" value="81" x="40.64" y="60.96" size="1.778" layer="27" rot="R180" display="off"/>

Commit message: Add files via upload
Parts:
- moved R1 5.24 mm to (45.7, 62.2), turned to 90 degrees
- moved X2 2.54 mm to (62.2, 47.0)
Connections:
- removed net N$8: T1.1, X2.1
- net N$2: now also X2.1
- net N$6: now also T1.1
Routing:
- net N$6: track 22.2 -> 86.7 mm
- net N$2: track 37.1 -> 74.7 mm
- net N$8: track 10.7 -> 0.00 mm
- net N$3: track 11.1 -> 7.77 mm
- net N$9: track 8.89 -> 11.4 mm
Changed lines of the file:
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@@
 <attribute name="POPULARITY" value="40" x="34.29" y="104.14" size="1.778" layer="27" rot="R90" display="off"/>
 </element>
-<element name="X2" library="con-molex" library_urn="urn:adsk.eagle:library:165" package="22-23-2021" package3d_urn="urn:adsk.eagle:package:8078633/1" value="22-23-2021" x="59.69" y="46.99" smashed="yes" rot="R270">
-<attribute name="MF" value="MOLEX" x="31.75" y="8.89" size="1.778" layer="27" rot="R270" display="off"/>
-<attribute name="MPN" value="22-23-2021" x="31.75" y="8.89" size="1.778" layer="27" rot="R270" display="off"/>
-<attribute name="NAME" x="63.5" y="49.53" size="1.016" layer="25" ratio="10" rot="R270"/>
-<attribute name="OC_FARNELL" value="1462926" x="31.75" y="8.89" size="1.778" layer="27" rot="R270" display="off"/>
-<attribute name="OC_NEWARK" value="25C3832" x="31.75" y="8.89" size="1.778" layer="27" rot="R270" display="off"/>
-<attribute name="POPULARITY" value="40" x="31.75" y="8.89" size="1.778" layer="27" rot="R270" display="off"/>
-<attribute name="VALUE" x="54.61" y="49.53" size="1.016" layer="27" ratio="10" rot="R270"/>
+<element name="X2" library="con-molex" library_urn="urn:adsk.eagle:library:165" package="22-23-2021" package3d_urn="urn:adsk.eagle:package:8078633/1" value="22-23-2021" x="62.23" y="46.99" smashed="yes" rot="R270">
+<attribute name="MF" value="MOLEX" x="34.29" y="8.89" size="1.778" layer="27" rot="R270" display="off"/>
+<attribute name="MPN" value="22-23-2021" x="34.29" y="8.89" size="1.778" layer="27" rot="R270" display="off"/>
+<attribute name="NAME" x="66.04" y="49.53" size="1.016" layer="25" ratio="10" rot="R270"/>
+<attribute name="OC_FARNELL" value="1462926" x="34.29" y="8.89" size="1.778" layer="27" rot="R270" display="off"/>
+<attribute name="OC_NEWARK" value="25C3832" x="34.29" y="8.89" size="1.778" layer="27" rot="R270" display="off"/>
+<attribute name="POPULARITY" value="40" x="34.29" y="8.89" size="1.778" layer="27" rot="R270" display="off"/>
+<attribute name="VALUE" x="57.15" y="49.53" size="1.016" layer="27" ratio="10" rot="R270"/>
 </element>
 <element name="T1" library="transistor-neu-to92" library_urn="urn:adsk.eagle:library:397" package="TO92" package3d_urn="urn:adsk.eagle:package:28725/2" value="2N3904" x="50.8" y="46.99" smashed="yes" rot="R90">
@@
 <attribute name="VALUE" x="19.685" y="54.3306" size="1.27" layer="27" ratio="10" rot="R270"/>
 </element>
-<element name="R1" library="rcl" library_urn="urn:adsk.eagle:library:334" package="0207/10" package3d_urn="urn:adsk.eagle:package:23491/2" value="5k6" x="40.64" y="60.96" smashed="yes" rot="R180">
-<attribute name="NAME" x="43.688" y="59.436" size="1.27" layer="25" ratio="10" rot="R180"/>
-<attribute name="POPULARITY" value="81" x="40.64" y="60.96" size="1.778" layer="27" rot="R180" display="off"/>
-<attribute name="SPICEPREFIX" value="R" x="40.64" y="60.96" size="1.778" layer="27" rot="R180" display="off"/>
-<attribute name="VALUE" x="42.9006" y="61.595" size="1.27" layer="27" ratio="10" rot="R180"/>
+<element name="R1" library="rcl" library_urn="urn:adsk.eagle:library:334" package="0207/10" package3d_urn="urn:adsk.eagle:package:23491/2" value="5k6" x="45.72" y="62.23" smashed="yes" rot="R90">
+<attribute name="NAME" x="44.196" y="59.182" size="1.27" layer="25" ratio="10" rot="R90"/>
+<attribute name="POPULARITY" value="81" x="45.72" y="62.23" size="1.778" layer="27" rot="R90" display="off"/>
+<attribute name="SPICEPREFIX" value="R" x="45.72" y="62.23" size="1.778" layer="27" rot="R90" display="off"/>
+<attribute name="VALUE" x="46.355" y="59.9694" size="1.27" layer="27" ratio="10" rot="R90"/>
 </element>
 </elements>
@@
 <wire x1="27.94" y1="61.976" x2="27.94" y2="62.23" width="0.508" layer="16"/>
 <contactref element="R1" pad="2"/>
-<wire x1="32.004" y1="60.96" x2="35.56" y2="60.96" width="0.508" layer="16"/>
+<wire x1="32.004" y1="60.96" x2="45.72" y2="67.31" width="0.508" layer="16"/>
 <wire x1="30.48" y1="59.436" x2="32.004" y2="60.96" width="0.508" layer="16"/>
+<contactref element="X2" pad="1"/>
+<wire x1="61.976" y1="50.8" x2="61.976" y2="48.26" width="0.508" layer="16"/>
+<wire x1="45.72" y1="67.056" x2="61.976" y2="50.8" width="0.508" layer="16"/>
+<wire x1="61.976" y1="48.26" x2="62.23" y2="48.26" width="0.508" layer="16"/>
+<wire x1="45.72" y1="67.056" x2="45.72" y2="67.31" width="0.508" layer="16"/>
 </signal>
 <signal name="N$6">
@@
 <wire x1="20.32" y1="59.944" x2="20.32" y2="57.15" width="0.508" layer="16"/>
 <wire x1="22.86" y1="62.484" x2="20.32" y2="59.944" width="0.508" layer="16"/>
+<contactref element="T1" pad="1"/>
+<wire x1="49.784" y1="48.26" x2="50.8" y2="48.26" width="0.508" layer="16"/>
+<wire x1="48.768" y1="49.276" x2="49.784" y2="48.26" width="0.508" layer="16"/>
+<wire x1="40.132" y1="49.276" x2="48.768" y2="49.276" width="0.508" layer="16"/>
+<wire x1="38.608" y1="47.752" x2="40.132" y2="49.276" width="0.508" layer="16"/>
+<wire x1="38.608" y1="46.228" x2="38.608" y2="47.752" width="0.508" layer="16"/>
+<wire x1="40.64" y1="44.196" x2="38.608" y2="46.228" width="0.508" layer="16"/>
+<wire x1="41.148" y1="44.196" x2="40.64" y2="44.196" width="0.508" layer="16"/>
+<wire x1="42.672" y1="42.672" x2="41.148" y2="44.196" width="0.508" layer="16"/>
+<wire x1="42.672" y1="41.148" x2="42.672" y2="42.672" width="0.508" layer="16"/>
+<wire x1="40.64" y1="39.116" x2="42.672" y2="41.148" width="0.508" layer="16"/>
+<wire x1="20.828" y1="39.116" x2="40.64" y2="39.116" width="0.508" layer="16"/>
+<wire x1="18.288" y1="41.656" x2="20.828" y2="39.116" width="0.508" layer="16"/>
+<wire x1="18.288" y1="54.864" x2="18.288" y2="41.656" width="0.508" layer="16"/>
+<wire x1="20.32" y1="56.896" x2="18.288" y2="54.864" width="0.508" layer="16"/>
+<wire x1="20.32" y1="56.896" x2="20.32" y2="57.15" width="0.508" layer="16"/>
 </signal>
 <signal name="N$7">
@@
 <contactref element="R2" pad="1"/>
 <contactref element="R1" pad="1"/>
-<wire x1="45.72" y1="57.404" x2="45.72" y2="60.96" width="0.508" layer="16"/>
+<wire x1="45.72" y1="57.404" x2="45.72" y2="57.15" width="0.508" layer="16"/>
 <wire x1="40.64" y1="52.324" x2="45.72" y2="57.404" width="0.508" layer="16"/>
 <wire x1="40.64" y1="52.324" x2="40.64" y2="51.99" width="0.508" layer="16"/>
@@
 <wire x1="40.64" y1="47.244" x2="40.64" y2="46.99" width="0.508" layer="16"/>
 </signal>
-<signal name="N$8">
-<contactref element="T1" pad="1"/>
-<contactref element="X2" pad="1"/>
-<wire x1="59.182" y1="48.768" x2="51.054" y2="48.768" width="1.016" layer="16"/>
-<wire x1="51.054" y1="48.768" x2="49.784" y2="48.768" width="1.016" layer="16"/>
-<wire x1="51.054" y1="48.768" x2="50.8" y2="48.26" width="1.016" layer="16"/>
-<wire x1="59.182" y1="48.768" x2="59.69" y2="48.26" width="1.016" layer="16"/>
-</signal>
 <signal name="N$9">
 <contactref element="T1" pad="3"/>
 <contactref element="X2" pad="2"/>
-<wire x1="59.69" y1="45.72" x2="50.8" y2="45.72" width="1.016" layer="16"/>
+<wire x1="62.23" y1="45.72" x2="50.8" y2="45.72" width="1.016" layer="16"/>
 </signal>
 </signals>

Commit message: Add files via upload
Parts:
- R1: value 5k6 -> 5k2
- moved X2 37.8 mm to (36.8, 74.9), turned to 0 degrees
- moved R1 25.0 mm to (21.6, 55.9), turned to 180 degrees
- moved D1 20.5 mm to (35.6, 59.7), turned to 90 degrees
- moved T1 20.1 mm to (44.5, 66.0), turned to 0 degrees
- moved R4 17.6 mm to (11.4, 67.3)
- moved C1 13.0 mm to (29.2, 74.9), turned to 270 degrees
- moved R2 4.58 mm to (38.1, 50.8), turned to 0 degrees
- moved B1 1.27 mm to (19.1, 69.8)
Routing:
- net N$9: track 11.4 -> 96.6 mm
- net N$6: track 86.7 -> 46.0 mm
- net N$4: track 27.3 -> 40.8 mm
- net N$5: track 10.4 -> 20.6 mm
- net N$2: track 74.7 -> 65.1 mm
- net N$1: track 15.7 -> 19.2 mm
- net N$7: track 11.7 -> 12.8 mm
- net N$3: track 7.77 -> 8.53 mm
