File: fonte.sch (EAGLE design)
At the start: 9 parts, among them T1 2N3904, X1 22-23-2021, X2 22-23-2021

Commit message: Add files via upload
Parts:
- R1: value 2k -> 5k6
- R2: value 4k7 -> 10k
- R4: value 200R -> 2k2
Changed lines of the file:
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@@
 <part name="B1" library="rectifier" library_urn="urn:adsk.eagle:library:336" deviceset="1KAB" device="" package3d_urn="urn:adsk.eagle:package:23872/1" value="20V"/>
 <part name="C1" library="rcl" library_urn="urn:adsk.eagle:library:334" deviceset="CPOL-EU" device="E2,5-6E" package3d_urn="urn:adsk.eagle:package:23430/1" value="470uF"/>
-<part name="R2" library="pot" library_urn="urn:adsk.eagle:library:331" deviceset="3RP/1610N" device="" package3d_urn="urn:adsk.eagle:package:22726/1" value="4k7"/>
+<part name="R2" library="pot" library_urn="urn:adsk.eagle:library:331" deviceset="3RP/1610N" device="" package3d_urn="urn:adsk.eagle:package:22726/1" value="10k"/>
 <part name="T1" library="transistor-neu-to92" library_urn="urn:adsk.eagle:library:397" deviceset="2N3904" device="" package3d_urn="urn:adsk.eagle:package:28725/2"/>
 <part name="D1" library="diode" library_urn="urn:adsk.eagle:library:210" deviceset="1N4728" device="" package3d_urn="urn:adsk.eagle:package:43341/1"/>
-<part name="R4" library="rcl" library_urn="urn:adsk.eagle:library:334" deviceset="R-EU_" device="0207/10" package3d_urn="urn:adsk.eagle:package:23491/2" value="200R"/>
-<part name="R1" library="rcl" library_urn="urn:adsk.eagle:library:334" deviceset="R-EU_" device="0207/10" package3d_urn="urn:adsk.eagle:package:23491/2" value="2k"/>
+<part name="R4" library="rcl" library_urn="urn:adsk.eagle:library:334" deviceset="R-EU_" device="0207/10" package3d_urn="urn:adsk.eagle:package:23491/2" value="2k2"/>
+<part name="R1" library="rcl" library_urn="urn:adsk.eagle:library:334" deviceset="R-EU_" device="0207/10" package3d_urn="urn:adsk.eagle:package:23491/2" value="5k6"/>
 </parts>
 <sheets>

Commit message: Add files via upload
Connections:
- removed net N$8: T1.C, X2-1.S
- net N$2: now also X2-1.S
- net N$6: now also T1.C
Other:
- moved on the sheet: X2-1, X2-2
Changed lines of the file:
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@@
 <attribute name="NAME" x="-12.7" y="87.122" size="1.524" layer="95" rot="R180"/>
 </instance>
-<instance part="X2" gate="-1" x="129.54" y="101.6" smashed="yes">
-<attribute name="NAME" x="132.08" y="100.838" size="1.524" layer="95"/>
+<instance part="X2" gate="-1" x="116.84" y="81.28" smashed="yes">
+<attribute name="NAME" x="119.38" y="80.518" size="1.524" layer="95"/>
 </instance>
-<instance part="X2" gate="-2" x="129.54" y="99.06" smashed="yes">
-<attribute name="NAME" x="132.08" y="98.298" size="1.524" layer="95"/>
+<instance part="X2" gate="-2" x="116.84" y="83.82" smashed="yes">
+<attribute name="NAME" x="119.38" y="83.058" size="1.524" layer="95"/>
 </instance>
 <instance part="B1" gate="1" x="20.32" y="88.9" smashed="yes">
@@
 <junction x="68.58" y="68.58"/>
 <pinref part="R1" gate="G$1" pin="2"/>
+<pinref part="X2" gate="-1" pin="S"/>
+<wire x1="114.3" y1="81.28" x2="106.68" y2="81.28" width="0.1524" layer="91"/>
+<wire x1="106.68" y1="81.28" x2="106.68" y2="68.58" width="0.1524" layer="91"/>
+<wire x1="106.68" y1="68.58" x2="81.28" y2="68.58" width="0.1524" layer="91"/>
+<junction x="81.28" y="68.58"/>
 </segment>
 </net>
@@
 <junction x="35.56" y="101.6"/>
 <pinref part="R4" gate="G$1" pin="1"/>
+<junction x="68.58" y="101.6"/>
+<wire x1="68.58" y1="101.6" x2="106.68" y2="101.6" width="0.1524" layer="91"/>
+<pinref part="T1" gate="G1" pin="C"/>
+<wire x1="106.68" y1="101.6" x2="106.68" y2="93.98" width="0.1524" layer="91"/>
 </segment>
 </net>
@@
 </segment>
 </net>
-<net name="N$8" class="0">
-<segment>
-<pinref part="T1" gate="G1" pin="C"/>
-<pinref part="X2" gate="-1" pin="S"/>
-<wire x1="106.68" y1="93.98" x2="106.68" y2="101.6" width="0.1524" layer="91"/>
-<wire x1="106.68" y1="101.6" x2="127" y2="101.6" width="0.1524" layer="91"/>
-</segment>
-</net>
 <net name="N$9" class="0">
 <segment>
 <pinref part="T1" gate="G1" pin="E"/>
-<wire x1="106.68" y1="83.82" x2="127" y2="83.82" width="0.1524" layer="91"/>
+<wire x1="106.68" y1="83.82" x2="114.3" y2="83.82" width="0.1524" layer="91"/>
 <pinref part="X2" gate="-2" pin="S"/>
-<wire x1="127" y1="83.82" x2="127" y2="99.06" width="0.1524" layer="91"/>
 </segment>
 </net>

Commit message: Add files via upload
Parts:
- R1: value 5k6 -> 5k2
Changed lines of the file:
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@@
 <part name="D1" library="diode" library_urn="urn:adsk.eagle:library:210" deviceset="1N4728" device="" package3d_urn="urn:adsk.eagle:package:43341/1"/>
 <part name="R4" library="rcl" library_urn="urn:adsk.eagle:library:334" deviceset="R-EU_" device="0207/10" package3d_urn="urn:adsk.eagle:package:23491/2" value="2k2"/>
-<part name="R1" library="rcl" library_urn="urn:adsk.eagle:library:334" deviceset="R-EU_" device="0207/10" package3d_urn="urn:adsk.eagle:package:23491/2" value="5k6"/>
+<part name="R1" library="rcl" library_urn="urn:adsk.eagle:library:334" deviceset="R-EU_" device="0207/10" package3d_urn="urn:adsk.eagle:package:23491/2" value="5k2"/>
 </parts>
 <sheets>
